Commit message: added and converted from .urdf to xacro

File: urdf/robot.xacro (robot description, xacro)
@@ -1,47 +1,5 @@
 <?xml version="1.0" ?>
-<robot name="robot">
-<gazebo reference="joint_chassis_caster_wheel">
-    <preserveFixedJoint>true</preserveFixedJoint>
-</gazebo>
-    <gazebo reference="link_chassis">
-        <material>Gazebo/Blue</material>
-    </gazebo>
-    <gazebo reference="link_left_wheel">
-        <material>Gazebo/Black</material>
-        <mu1>1</mu1>
-        <mu2>1</mu2>
-    </gazebo>
-    <gazebo reference="link_right_wheel">
-        <material>Gazebo/Black</material>
-        <mu1>1</mu1>
-        <mu2>1</mu2>
-    </gazebo>
-    <gazebo reference="link_caster_wheel">
-        <material>Gazebo/CloudySky</material>
-        <mu1>0</mu1>
-        <mu2>0</mu2>
-    </gazebo>
-    <gazebo>
-        <plugin filename="libgazebo_ros_diff_drive.so" name="differential_drive_controller">
-            <alwaysOn>true</alwaysOn>
-            <updateRate>20</updateRate>
-            <leftJoint>joint_chassis_left_wheel</leftJoint>
-            <rightJoint>joint_chassis_right_wheel</rightJoint>
-            <wheelSeparation>1.66</wheelSeparation>
-            <wheelDiameter>0.8</wheelDiameter>
-            <torque>10</torque>
-            <commandTopic>cmd_vel</commandTopic>
-            <odometryTopic>odom</odometryTopic>
-            <odometryFrame>odom</odometryFrame>
-            <robotBaseFrame>link_chassis</robotBaseFrame>
-        </plugin>
-    </gazebo>
-    <!-- Gazebo tags - Laser scan -->
-    <gazebo reference="joint_laser_scan_chassis">
-        <preserveFixedJoint>true</preserveFixedJoint>
-    </gazebo>
-    <gazebo reference="link_laser_scan">
-        <material>Gazebo/DarkGrey</material>
-    </gazebo>
+<robot name="robot" xmlns:xacro="http://www.ros.org/wiki/xacro">
+    <xacro:include filename="$(find robot_description)/urdf/robot.gazebo"/>
     <!-- Laser scan -->
     <joint name="joint_laser_scan_chassis" type="fixed">
@@ -73,35 +31,4 @@
         </collision>
     </link>
-    <gazebo reference="link_laser_scan">
-        <sensor type="ray" name="head_hokuyo_sensor">
-            <pose>0 0 0 0 0 0</pose>
-            <visualize>true</visualize>
-            <update_rate>20</update_rate>
-            <ray>
-                <scan>
-                    <horizontal>
-                        <samples>720</samples>
-                        <resolution>1</resolution>
-                        <min_angle>-1.570796</min_angle>
-                        <max_angle>1.570796</max_angle>
-                    </horizontal>
-                </scan>
-                <range>
-                    <min>0.20</min>
-                    <max>10.0</max>
-                    <resolution>0.01</resolution>
-                </range>
-                <noise>
-                    <type>gaussian</type>
-                    <mean>0.0</mean>
-                    <stddev>0.01</stddev>
-                </noise>
-            </ray>
-            <plugin name="gazebo_ros_head_hokuyo_controller" filename="libgazebo_ros_laser.so">
-                <topicName>/laser/scan</topicName>
-                <frameName>sensor_laser</frameName>
-            </plugin>
-        </sensor>
-    </gazebo>
     <!-- Link - chassis -->
     <link name="link_chassis">

Commit message: added xacro parameters (pi and chassis mass)

File: urdf/robot.xacro (robot description, xacro)
@@ -2,4 +2,7 @@
 <robot name="robot" xmlns:xacro="http://www.ros.org/wiki/xacro">
     <xacro:include filename="$(find robot_description)/urdf/robot.gazebo"/>
+    <!-- parameters -->
+    <xacro:property name="chassis_mass" value="10"/>
+    <xacro:property name="pi" value="3.14159265359"/>
     <!-- Laser scan -->
     <joint name="joint_laser_scan_chassis" type="fixed">
@@ -34,5 +37,5 @@
     <link name="link_chassis">
         <inertial>
-            <mass value="10" />
+            <mass value="${chassis_mass}" />
             <origin xyz="0 0 0.3" rpy="0 0 0" />
             <inertia ixx="1.5417" ixy="0" ixz="0" iyy="3.467" iyz="0" izz="4.742" />
@@ -69,11 +72,11 @@
     </inertial>
     <collision>
-        <origin rpy="1.5707 0 0" xyz="0 0.18 0" />
-        <geometry>
-            <mesh filename="package://robot_description/meshes/wheel.stl"/>
-        </geometry>
-    </collision>
-    <visual>
-        <origin rpy="1.5707 0 0" xyz="0 0.18 0" />
+        <origin rpy="${pi/2} 0 0" xyz="0 0.18 0" />
+        <geometry>
+            <mesh filename="package://robot_description/meshes/wheel.stl"/>
+        </geometry>
+    </collision>
+    <visual>
+        <origin rpy="${pi/2} 0 0" xyz="0 0.18 0" />
         <geometry>
             <mesh filename="package://robot_description/meshes/wheel.stl"/>
@@ -84,5 +87,5 @@
     </visual>
     <collision>
-        <origin rpy="1.5707 0 0" xyz="0 0.06 0" />
+        <origin rpy="${pi/2} 0 0" xyz="0 0.06 0" />
         <geometry>
             <cylinder length="0.12" radius="0.08"/>
@@ -90,5 +93,5 @@
     </collision>
     <visual>
-        <origin rpy="1.5707 0 0" xyz="0 0.06 0" />
+        <origin rpy="${pi/2} 0 0" xyz="0 0.06 0" />
         <geometry>
             <cylinder length="0.16" radius="0.08"/>
@@ -131,11 +134,11 @@
     </inertial>
     <collision>
-        <origin rpy="1.5707 0 0" xyz="0 -0.18 0" />
-        <geometry>
-            <mesh filename="package://robot_description/meshes/wheel.stl"/>
-        </geometry>
-    </collision>
-    <visual>
-        <origin rpy="1.5707 0 0" xyz="0 -0.18 0" />
+        <origin rpy="${pi/2} 0 0" xyz="0 -0.18 0" />
+        <geometry>
+            <mesh filename="package://robot_description/meshes/wheel.stl"/>
+        </geometry>
+    </collision>
+    <visual>
+        <origin rpy="${pi/2} 0 0" xyz="0 -0.18 0" />
         <geometry>
             <mesh filename="package://robot_description/meshes/wheel.stl"/>
@@ -146,5 +149,5 @@
     </visual>
     <collision>
-        <origin rpy="1.5707 0 0" xyz="0 -0.06 0" />
+        <origin rpy="${pi/2} 0 0" xyz="0 -0.06 0" />
         <geometry>
             <cylinder length="0.18" radius="0.08"/>
@@ -152,5 +155,5 @@
     </collision>
     <visual>
-        <origin rpy="1.5707 0 0" xyz="0 -0.06 0" />
+        <origin rpy="${pi/2} 0 0" xyz="0 -0.06 0" />
         <geometry>
             <cylinder length="0.18" radius="0.08"/>

Commit message: added tail

File: urdf/robot.xacro (robot description, xacro)
@@ -5,4 +5,237 @@
     <xacro:property name="chassis_mass" value="10"/>
     <xacro:property name="pi" value="3.14159265359"/>
+    <!-- Link - chassis -->
+    <link name="link_chassis">
+        <inertial>
+            <mass value="${chassis_mass}" />
+            <origin xyz="0 0 0.3" rpy="0 0 0" />
+            <inertia ixx="1.5417" ixy="0" ixz="0" iyy="3.467" iyz="0" izz="4.742" />
+        </inertial>
+        <collision>
+            <geometry>
+                <mesh filename="package://robot_description/meshes/chassis.stl" />
+            </geometry>
+        </collision>
+        <visual>
+            <geometry>
+                <mesh filename="package://robot_description/meshes/chassis.stl" />
+            </geometry>
+            <material name="Blue">
+                <color rgba="0 0 1 1" />
+            </material>
+        </visual>
+    </link>
+<!-- Joint - chassis / left wheel -->
+<joint name="joint_chassis_left_wheel" type="continuous">
+    <origin rpy="0 0 0" xyz="-0.5 0.65 0" />
+    <child link="link_left_wheel" />
+    <parent link="link_chassis" />
+    <axis rpy="0 0 0" xyz="0 1 0" />
+    <limit effort="10000" velocity="1000" />
+    <joint_properties damping="1.0" friction="1.0" />
+</joint>
+<!-- Link - left wheel -->
+<link name="link_left_wheel">
+    <inertial>
+        <mass value="1" />
+        <origin xyz="0 0 0" rpy="0 0 0" />
+        <inertia ixx="0.002526666666667" ixy="0" ixz="0" iyy="0.002526666666667" iyz="0" izz="0.005"/>
+    </inertial>
+    <collision>
+        <origin rpy="${pi/2} 0 0" xyz="0 0.18 0" />
+        <geometry>
+            <mesh filename="package://robot_description/meshes/wheel.stl"/>
+        </geometry>
+    </collision>
+    <visual>
+        <origin rpy="${pi/2} 0 0" xyz="0 0.18 0" />
+        <geometry>
+            <mesh filename="package://robot_description/meshes/wheel.stl"/>
+        </geometry>
+        <material name="black">
+            <color rgba="0 0 0 1" />
+        </material>
+    </visual>
+    <collision>
+        <origin rpy="${pi/2} 0 0" xyz="0 0.06 0" />
+        <geometry>
+            <cylinder length="0.12" radius="0.08"/>
+        </geometry>
+    </collision>
+    <visual>
+        <origin rpy="${pi/2} 0 0" xyz="0 0.06 0" />
+        <geometry>
+            <cylinder length="0.16" radius="0.08"/>
+        </geometry>
+        <material name="white">
+            <color rgba="1 1 1 1" />
+        </material>
+    </visual>
+    <collision>
+        <origin rpy="0 0 0" xyz="0 0.17 0"/>
+        <geometry>
+            <box size="0.05 0.1 0.6"/>
+        </geometry>
+    </collision>
+    <visual>
+        <origin rpy="0 0 0" xyz="0 0.17 0"/>
+        <geometry>
+           <box size="0.05 0.10 0.6"/>
+        </geometry>
+        <material name="white">
+            <color rgba="1 1 1 1" />
+        </material>
+    </visual>
+</link>
+<!-- Joint - chassis / right wheel -->
+<joint name="joint_chassis_right_wheel" type="continuous">
+    <origin rpy="0 0 0" xyz="-0.5 -0.65 0" />
+    <child link="link_right_wheel" />
+    <parent link="link_chassis" />
+    <axis rpy="0 0 0" xyz="0 1 0" />
+   <limit effort="10000" velocity="1000" />
+    <joint_properties damping="1.0" friction="1.0" />
+</joint>
+<!-- Link - right wheel -->
+<link name="link_right_wheel">
+    <inertial>
+        <mass value="1" />
+        <origin xyz="0 0 0" rpy="0 0 0" />
+        <inertia ixx="0.002526666666667" ixy="0" ixz="0" iyy="0.002526666666667" iyz="0" izz="0.005"/>
+    </inertial>
+    <collision>
+        <origin rpy="${pi/2} 0 0" xyz="0 -0.18 0" />
+        <geometry>
+            <mesh filename="package://robot_description/meshes/wheel.stl"/>
+        </geometry>
+    </collision>
+    <visual>
+        <origin rpy="${pi/2} 0 0" xyz="0 -0.18 0" />
+        <geometry>
+            <mesh filename="package://robot_description/meshes/wheel.stl"/>
+        </geometry>
+        <material name="black">
+               <color rgba="0 0 0 1" />
+        </material>
+    </visual>
+    <collision>
+        <origin rpy="${pi/2} 0 0" xyz="0 -0.06 0" />
+        <geometry>
+            <cylinder length="0.18" radius="0.08"/>
+        </geometry>
+    </collision>
+    <visual>
+        <origin rpy="${pi/2} 0 0" xyz="0 -0.06 0" />
+        <geometry>
+            <cylinder length="0.18" radius="0.08"/>
+        </geometry>
+        <material name="white">
+            <color rgba="1 1 1 1" />
+        </material>
+    </visual>
+    <collision>
+        <origin rpy="0 0 0" xyz="0 -0.17 0"/>
+        <geometry>
+            <box size="0.05 0.1 0.6"/>
+        </geometry>
+    </collision>
+    <visual>
+        <origin rpy="0 0 0" xyz="0 -0.17 0"/>
+        <geometry>
+           <box size="0.05 0.10 0.6"/>
+        </geometry>
+        <material name="white">
+            <color rgba="1 1 1 1" />
+        </material>
+    </visual>
+</link>
+<!-- joint chassis/robot_tail -->
+<joint name="joint_tail" type="continuous">
+    <origin rpy="0 0 0" xyz="-1 0 0"/>
+    <child link="link_tail"/>
+    <parent link="link_chassis"/>
+    <axis rpy="0 0 0" xyz="0 1 0"/>
+    <joint_properties damping="1.0" friction="1.0"/>
+</joint>
+<!-- link tail -->
+<link name="link_tail">
+    <inertial>
+        <origin xyz="0 0 0" rpy="0 0 0"/>
+        <mass value="0.5"/>
+        <inertia ixx="0.000252666666667" ixy="0" ixz="0" iyy="0.000252666666667" iyz="0" izz="0.0005"/>
+    </inertial>
+    <collision>
+        <origin xyz="-0.2 0 0" rpy="0 ${pi/2} 0"/>
+        <geometry>
+            <cylinder radius="0.05" length="0.4"/>
+        </geometry>
+    </collision>
+    <visual>
+        <origin xyz="-0.2 0 0" rpy="0 ${pi/2} 0"/>
+        <geometry>
+            <cylinder radius="0.05" length="0.4"/>
+        </geometry>
+        <material name="Red">
+            <color rgba="0.7 0.1 0.1 1"/>
+        </material>
+    </visual>
+</link>
+<transmission name="tran_tail">
+    <type>transmission_interface/SimpleTransmission</type>
+    <joint name="joint_tail">
+        <hardwareInterface>hardware_interface/EffortJointInterface</hardwareInterface>
+    </joint>
+    <actuator name="motor_joint_tail">
+        <hardwareInterface>hardware_interface/EffortJointInterface</hardwareInterface>
+        <mechanicalReduction>1</mechanicalReduction>
+    </actuator>
+</transmission>
+<!-- joint chassis/caster wheel -->
+<joint name="joint_chassis_caster_wheel" type="fixed">
+    <origin rpy="0 0 0" xyz="0.75 0 -0.15"/>
+    <child link="link_caster_wheel"/>
+    <parent link="link_chassis"/>
+    <axis rpy="0 0 0" xyz="1 1 1"/>
+    <limit effort="10000" velocity="1000" />
+    <joint_properties damping="1.0" friction="1.0" />
+</joint>
+<!-- link caster wheel -->
+<link name="link_caster_wheel">
+    <inertial>
+        <mass value="0.5"/>
+        <origin rpy="0 0 0" xyz="0 0 0"/>
+        <inertia ixx="0.002526666666667" ixy="0" ixz="0" iyy="0.002526666666667" iyz="0" izz="0.005"/>
+    </inertial>
+    <collision>
+        <origin rpy="0 0 0" xyz="0 0 0"/>
+        <geometry>
+            <sphere radius="0.25"/>
+        </geometry>
+    </collision>
+    <visual>
+        <origin rpy="0 0 0" xyz="0 0 0"/>
+        <geometry>
+            <sphere radius="0.25"/>
+        </geometry>
+        <material name="blue">
+                <color rgba="0 0 1 1" />
+        </material>
+    </visual>
+<collision>
+        <origin rpy="0 0 0" xyz="0 0 -0.156"/>
+        <geometry>
+            <sphere radius="0.125"/>
+        </geometry>
+    </collision>
+    <visual>
+        <origin rpy="0 0 0" xyz="0 0 -0.156"/>
+        <geometry>
+            <sphere radius="0.125"/>
+        </geometry>
+        <material name="white">
+            <color rgba="1 1 1 1" />
+        </material>
+    </visual>
+</link>
     <!-- Laser scan -->
     <joint name="joint_laser_scan_chassis" type="fixed">
@@ -34,195 +267,3 @@
         </collision>
     </link>
-    <!-- Link - chassis -->
-    <link name="link_chassis">
-        <inertial>
-            <mass value="${chassis_mass}" />
-            <origin xyz="0 0 0.3" rpy="0 0 0" />
-            <inertia ixx="1.5417" ixy="0" ixz="0" iyy="3.467" iyz="0" izz="4.742" />
-        </inertial>
-        <collision>
-            <geometry>
-                <mesh filename="package://robot_description/meshes/chassis.stl" />
-            </geometry>
-        </collision>
-        <visual>
-            <geometry>
-                <mesh filename="package://robot_description/meshes/chassis.stl" />
-            </geometry>
-            <material name="Blue">
-                <color rgba="0 0 1 1" />
-            </material>
-        </visual>
-    </link>
-<!-- Joint - chassis / left wheel -->
-<joint name="joint_chassis_left_wheel" type="continuous">
-    <origin rpy="0 0 0" xyz="-0.5 0.65 0" />
-    <child link="link_left_wheel" />
-    <parent link="link_chassis" />
-    <axis rpy="0 0 0" xyz="0 1 0" />
-    <limit effort="10000" velocity="1000" />
-    <joint_properties damping="1.0" friction="1.0" />
-</joint>
-<!-- Link - left wheel -->
-<link name="link_left_wheel">
-    <inertial>
-        <mass value="1" />
-        <origin xyz="0 0 0" rpy="0 0 0" />
-        <inertia ixx="0.002526666666667" ixy="0" ixz="0" iyy="0.002526666666667" iyz="0" izz="0.005"/>
-    </inertial>
-    <collision>
-        <origin rpy="${pi/2} 0 0" xyz="0 0.18 0" />
-        <geometry>
-            <mesh filename="package://robot_description/meshes/wheel.stl"/>
-        </geometry>
-    </collision>
-    <visual>
-        <origin rpy="${pi/2} 0 0" xyz="0 0.18 0" />
-        <geometry>
-            <mesh filename="package://robot_description/meshes/wheel.stl"/>
-        </geometry>
-        <material name="black">
-            <color rgba="0 0 0 1" />
-        </material>
-    </visual>
-    <collision>
-        <origin rpy="${pi/2} 0 0" xyz="0 0.06 0" />
-        <geometry>
-            <cylinder length="0.12" radius="0.08"/>
-        </geometry>
-    </collision>
-    <visual>
-        <origin rpy="${pi/2} 0 0" xyz="0 0.06 0" />
-        <geometry>
-            <cylinder length="0.16" radius="0.08"/>
-        </geometry>
-        <material name="white">
-            <color rgba="1 1 1 1" />
-        </material>
-    </visual>
-    <collision>
-        <origin rpy="0 0 0" xyz="0 0.17 0"/>
-        <geometry>
-            <box size="0.05 0.1 0.6"/>
-        </geometry>
-    </collision>
-    <visual>
-        <origin rpy="0 0 0" xyz="0 0.17 0"/>
-        <geometry>
-           <box size="0.05 0.10 0.6"/>
-        </geometry>
-        <material name="white">
-            <color rgba="1 1 1 1" />
-        </material>
-    </visual>
-</link>
-<!-- Joint - chassis / right wheel -->
-<joint name="joint_chassis_right_wheel" type="continuous">
-    <origin rpy="0 0 0" xyz="-0.5 -0.65 0" />
-    <child link="link_right_wheel" />
-    <parent link="link_chassis" />
-    <axis rpy="0 0 0" xyz="0 1 0" />
-   <limit effort="10000" velocity="1000" />
-    <joint_properties damping="1.0" friction="1.0" />
-</joint>
-<!-- Link - right wheel -->
-<link name="link_right_wheel">
-    <inertial>
-        <mass value="1" />
-        <origin xyz="0 0 0" rpy="0 0 0" />
-        <inertia ixx="0.002526666666667" ixy="0" ixz="0" iyy="0.002526666666667" iyz="0" izz="0.005"/>
-    </inertial>
-    <collision>
-        <origin rpy="${pi/2} 0 0" xyz="0 -0.18 0" />
-        <geometry>
-            <mesh filename="package://robot_description/meshes/wheel.stl"/>
-        </geometry>
-    </collision>
-    <visual>
-        <origin rpy="${pi/2} 0 0" xyz="0 -0.18 0" />
-        <geometry>
-            <mesh filename="package://robot_description/meshes/wheel.stl"/>
-        </geometry>
-        <material name="black">
-               <color rgba="0 0 0 1" />
-        </material>
-    </visual>
-    <collision>
-        <origin rpy="${pi/2} 0 0" xyz="0 -0.06 0" />
-        <geometry>
-            <cylinder length="0.18" radius="0.08"/>
-        </geometry>
-    </collision>
-    <visual>
-        <origin rpy="${pi/2} 0 0" xyz="0 -0.06 0" />
-        <geometry>
-            <cylinder length="0.18" radius="0.08"/>
-        </geometry>
-        <material name="white">
-            <color rgba="1 1 1 1" />
-        </material>
-    </visual>
-    <collision>
-        <origin rpy="0 0 0" xyz="0 -0.17 0"/>
-        <geometry>
-            <box size="0.05 0.1 0.6"/>
-        </geometry>
-    </collision>
-    <visual>
-        <origin rpy="0 0 0" xyz="0 -0.17 0"/>
-        <geometry>
-           <box size="0.05 0.10 0.6"/>
-        </geometry>
-        <material name="white">
-            <color rgba="1 1 1 1" />
-        </material>
-    </visual>
-</link>
-<!-- joint chassis/caster wheel -->
-<joint name="joint_chassis_caster_wheel" type="fixed">
-    <origin rpy="0 0 0" xyz="0.75 0 -0.15"/>
-    <child link="link_caster_wheel"/>
-    <parent link="link_chassis"/>
-    <axis rpy="0 0 0" xyz="1 1 1"/>
-    <limit effort="10000" velocity="1000" />
-    <joint_properties damping="1.0" friction="1.0" />
-</joint>
-<!-- link caster wheel -->
-<link name="link_caster_wheel">
-    <inertial>
-        <mass value="0.5"/>
-        <origin rpy="0 0 0" xyz="0 0 0"/>
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